File: KiCAD/BT-E6000/BMS.kicad_sch (KiCad schematic)
At the start: 276 parts, among them CN001 CN001, CN003 S04B-ZESK-2D_T__LF__SN_, CN004 S04B-ZESK-2D_T__LF__SN_, CN2 CN002, IC002 TPS7A1633DGNT, J1 -, J2 Rx, J3 Tx, J4 +, Q001 Q_PNP, Q002 Q_PNP, Q003 Q_PNP, Q004 Q_PNP, Q005 Q_PNP, Q006 ATP304-TL-H, Q007 ATP304-TL-H, Q008 ATP304-TL-H, Q009 ATP304-TL-H, Q010 ATP304-TL-H, Q011 ATP304-TL-H, Q013 Q_PNP, Q014 Q_NPN, Q015 Q_NPN, Q016 Q_NPN, Q017 Q_NPN, Q018 Q_NPN, Q019 Q_NPN, Q020 Q_NPN, Q021 Q_NPN, Q022 Q_NPN, Q023 Q_NPN, Q024 Q_NPN, Q025 Q_NPN, Q026 Q_PMOS, Q027 Q_PMOS, Q028 Q_PMOS, Q12 Q_PNP, Q29 Q_NMOS, U1 BQ77PL900DL

Commit message: Added BT-E80?? images
Parts:
- added Q30: Q_NMOS, symbol Device:Q_NMOS
Other:
- note added: "MOSFETS"
- note added: "PACK"
- note added: "PCB"
Changed lines of the file:
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@@
 		)
 	)
+	(text "PCB"
+		(exclude_from_sim no)
+		(at 270.51 34.29 0)
+		(effects
+			(font
+				(size 1.27 1.27)
+			)
+			(justify left)
+		)
+	)
 	(text "TURNS ON LDO FOR IC003 POWER\nTRIGGERD VIA RX HIGH OR IC003_PIN19"
 		(exclude_from_sim no)
@@
 		)
 	)
+	(text "PACK"
+		(exclude_from_sim no)
+		(at 243.84 34.036 0)
+		(effects
+			(font
+				(size 1.27 1.27)
+			)
+			(justify left)
+		)
+	)
 	(text "Data I/O voltage 3.3V"
 		(exclude_from_sim no)
@@
 		)
 	)
+	(text "MOSFETS"
+		(exclude_from_sim no)
+		(at 217.17 34.29 0)
+		(effects
+			(font
+				(size 1.27 1.27)
+			)
+			(justify left)
+		)
+	)
 	(text "DISABLE CHARGE"
 		(exclude_from_sim no)
@@
 	(wire
 		(pts
-			(xy 266.7 250.19) (xy 266.7 247.65)
+			(xy 266.7 247.65) (xy 266.7 250.19)
 		)
 		(stroke
@@
 			)
 		)
-		(property "Datasheet" ""
+		(property "Datasheet" "https://6197088.fs1.hubspotusercontent-na2.net/hubfs/6197088/TDS/SCP/SFK%20series_Datasheet.pdf"
 			(at 33.02 187.96 0)
 			(effects
@@
 					(unit 1)
 				)
+			)
+		)
+	)
+	(symbol
+		(lib_name "Q_NMOS_1")
+		(lib_id "Device:Q_NMOS")
+		(at 248.92 246.38 270)
+		(unit 1)
+		(exclude_from_sim no)
+		(in_bom yes)
+		(on_board yes)
+		(dnp no)
+		(fields_autoplaced yes)
+		(property "Reference" "Q30"
+			(at 248.92 252.73 90)
+			(effects
+				(font
+					(size 1.27 1.27)
+				)
+			)
+		)
+		(property "Value" "Q_NMOS"
+			(at 248.92 255.27 90)
+			(effects
+				(font
+					(size 1.27 1.27)
+				)
+			)
+		)
+		(property "Footprint" ""
+			(at 251.46 251.46 0)
+			(effects
+				(font
+					(size 1.27 1.27)
+				)
+				(hide yes)
+			)
+		)
+		(property "Datasheet" "~"
+			(at 248.92 246.38 0)
+			(effects
+				(font
+					(size 1.27 1.27)
+				)
+				(hide yes)
+			)
+		)
+		(property "Description" "N-MOSFET transistor"
+			(at 248.92 246.38 0)
+			(effects
+				(font
+					(size 1.27 1.27)
+				)
+				(hide yes)
+			)
+		)
+		(pin "S"
+		)
+		(pin "D"
+		)
+		(pin "G"
+		)
+		(instances
+			(project ""
+				(path "/4e6beee8-2dfa-4c94-aba5-d25855cc9658"
+					(reference "Q30")
+					(unit 1)
+				)
